Commit message: updated contoller package

File: install/bumperbot_description/share/bumperbot_description/urdf/bumperbot_gazebo.xacro (robot description, xacro)
@@ -1,4 +1,18 @@
 <?xml version="1.0"?>
 <robot name="bumperbot" xmlns:xacro="http://www.ros.org/wiki.xacro">
+    <transmission name="wheel_right_transmission">
+        <plugin>transmission_interface/SimpleTransmission</plugin>
+        <actuator name="wheel_right_motor" role="actuator_right"/>
+        <joint name="wheel_right_joint" role="joint_right">
+            <mechanical_reduction>1.0</mechanical_reduction>
+        </joint>
+    </transmission>
+    <transmission name="wheel_left_transmission">
+        <plugin>transmission_interface/SimpleTransmission</plugin>
+        <actuator name="wheel_left_motor" role="actuator_left"/>
+        <joint name="wheel_left_joint" role="joint_left">
+            <mechanical_reduction>1.0</mechanical_reduction>
+        </joint>
+    </transmission>
     <gazebo reference="wheel_right_link">
         <mu1>100000000000000.0</mu1>
@@ -41,3 +55,10 @@
         <!-- this is the direction of rotation -->
     </gazebo>
+    <gazebo>
+        <plugin filename="libgazebo_ros2_control.so" name="gazebo_ros2_control">
+            <robot_param>robot_description</robot_param>
+            <robot_param_node>robot_state_publisher</robot_param_node>
+            <parameters>$(find bumperbot_controller)/config/bumperbot_controllers.yaml</parameters>
+        </plugin>
+    </gazebo>
 </robot>

File: src/bumperbot_description/urdf/bumperbot_gazebo.xacro (robot description, xacro)
@@ -59,5 +59,5 @@
             <robot_param>robot_description</robot_param>
             <robot_param_node>robot_state_publisher</robot_param_node>
-            <parameters></parameters>
+            <parameters>$(find bumperbot_controller)/config/bumperbot_controllers.yaml</parameters>
         </plugin>
     </gazebo>
